Commit message: Slight changes to urdf and controller gains

File: Simulation/urdf/drone.urdf (robot description, URDF)
Before this commit: robot drone, 7 links, 6 joints
Links:
- link ball_bot: mass 0.002 -> 0.003
- link ball_top: mass 0.002 -> 0.003
- link base: mass 0.032 -> 0.036
Joints:
- joint base_to_bar: axis 1 0 0 -> 0 1 0
